File: hardware/acoustic-swarm-node/acoustic-swarm-node.kicad_sch (KiCad schematic)
At the start: 91 parts, among them J1 PIEZO/HV, J10 SWARM BFSK TX1, J11 ARM-SW (NC), J12 MODEM KONTAKTOR, J2 HIDROFON AFE, J3 AKUSTIK I2C, J4 SIZINTI PROBU, J5 AKUSTIK CH0 TX, J6 AKUSTIK CH1 TX, J7 AKUSTIK CH2 TX, J8 AKUSTIK CH3 TX, J9 SWARM BFSK TX0, Q1 AO3400A, Q2 BCP56-16, U1 LMR16006XDDCR, U2 AP2112K-3.3, U3 Teensy 4.1

Commit message: refactor: rename carrier project to acoustic-swarm-node and simplify docs
Other:
- title: Pelagos Deniz Tabani Akustik Dugum Karti -> Akustik Suru Dugum Karti

Commit message: Rev A acoustic node board, 192 kHz DSP chain and authenticated BFSK mesh
Hardware
- New netlist: always-on wake-up chain (MCP6042 60 dB + TLV7031 gating
  the LMR16006X enable), dual-gain hydrophone AFE (MCP6022, 40 kHz
  Sallen-Key), discrete piezo harvester, DRV8871 BFSK driver, switched
  battery divider and reed arming switch
- Board grows to 120x95 mm; Teensy pin map follows block placement
- Router: same-numbered pads are one target, reverse search and
  corridor waypoints for board-length nets, GND stitching routed last
- KiCad 9 support (kicad_env paths, multi-unit symbols, global labels);
  DRC 0 violations / 0 unconnected with schematic parity
- 3D renders and layout view under hardware/images

Firmware
- Streaming LOFAR (2 kHz) and DEMON (375 Hz) processors on 192 kHz
  dual-ADC DMA input, dual-gain channel selection
- Goertzel BFSK receiver with 4 timing lanes and out-of-band energy gate
- SipHash-2-4 tagged 20-byte mesh frame (replaces 16-bit FNV tag)
- PowerManager state machine around PWR_HOLD / wake latch
- Host tests: dsp, bfsk_modem, swarm_mesh, power_manager (ASan/UBSan)

Model
- dsp/node_model.py derives AFE response, sleep current and link budget
  from design.py values and checks them against firmware constants
Parts:
- removed BZ1: 5V aktif, Buzzer_Beeper:Buzzer_12x9.5RM7.6, symbol Device:Buzzer
- removed C10: 100nF, Capacitor_SMD:C_0603_1608Metric, symbol Device:C
- removed D10, D3: SS16, Diode_SMD:D_SMA, symbol Device:D_Schottky
- removed D11: KIRMIZI, LED_SMD:LED_0603_1608Metric, symbol Device:LED
- removed D12, D7: BZT52C3V3, Diode_SMD:D_SOD-123, symbol Device:D_Zener
- removed D4: B5819W, Diode_SMD:D_SOD-123, symbol Device:D_Schottky
- removed D5: YESIL, LED_SMD:LED_0603_1608Metric, symbol Device:LED
- removed D6: BAT54S, Package_TO_SOT_SMD:SOT-23, symbol Diode:BAT54S
- removed D8: 1N4148W, Diode_SMD:D_SOD-323, symbol Device:D
- removed D9: MAVI, LED_SMD:LED_0603_1608Metric, symbol Device:LED
- removed J10: SWARM BFSK TX1, Connector_JST:JST_XH_B3B-XH-A_1x03_P2.50mm_Vertical, symbol Connector_Generic:Conn_01x03
- removed J11: ARM-SW (NC), Connector_JST:JST_XH_B2B-XH-A_1x02_P2.50mm_Vertical, symbol Connector_Generic:Conn_01x02
- removed J12: MODEM KONTAKTOR, Connector_JST:JST_XH_B2B-XH-A_1x02_P2.50mm_Vertical, symbol Connector_Generic:Conn_01x02
- removed J2: HIDROFON AFE, Connector_JST:JST_XH_B3B-XH-A_1x03_P2.50mm_Vertical, symbol Connector_Generic:Conn_01x03
- removed J3: AKUSTIK I2C, Connector_JST:JST_XH_B4B-XH-A_1x04_P2.50mm_Vertical, symbol Connector_Generic:Conn_01x04
- removed J4: SIZINTI PROBU, Connector_JST:JST_XH_B2B-XH-A_1x02_P2.50mm_Vertical, symbol Connector_Generic:Conn_01x02
- removed J5: AKUSTIK CH0 TX, Connector_JST:JST_XH_B3B-XH-A_1x03_P2.50mm_Vertical, symbol Connector_Generic:Conn_01x03
- removed J6: AKUSTIK CH1 TX, Connector_JST:JST_XH_B3B-XH-A_1x03_P2.50mm_Vertical, symbol Connector_Generic:Conn_01x03
- removed J7: AKUSTIK CH2 TX, Connector_JST:JST_XH_B3B-XH-A_1x03_P2.50mm_Vertical, symbol Connector_Generic:Conn_01x03
- removed J8: AKUSTIK CH3 TX, Connector_JST:JST_XH_B3B-XH-A_1x03_P2.50mm_Vertical, symbol Connector_Generic:Conn_01x03
- removed J9: SWARM BFSK TX0, Connector_JST:JST_XH_B3B-XH-A_1x03_P2.50mm_Vertical, symbol Connector_Generic:Conn_01x03
- removed Q1: AO3400A, Package_TO_SOT_SMD:SOT-23, symbol Transistor_FET:AO3400A
- removed Q2: BCP56-16, Package_TO_SOT_SMD:SOT-223-3_TabPin2, symbol Transistor_BJT:BCP56
- removed U1: LMR16006XDDCR, Package_TO_SOT_SMD:SOT-23-6, symbol Regulator_Switching:LMR16006YQ
- removed U2: AP2112K-3.3, Package_TO_SOT_SMD:SOT-23-5, symbol Regulator_Linear:AP2112K-3.3
- removed U3: Teensy 4.1, stingray:Teensy4.1_Socket, symbol stingray:Teensy4.1
- added C15, C20, C24, C25: 1uF, Capacitor_SMD:C_0603_1608Metric, symbol Device:C
- added C16, C18, C19, C32, C35, C41: 100nF, Capacitor_SMD:C_0603_1608Metric, symbol Device:C
- added C17: 470nF, Capacitor_SMD:C_0603_1608Metric, symbol Device:C
- added C21: 100nF 25V, Capacitor_SMD:C_0603_1608Metric, symbol Device:C
- added C22, C23: 22uF 10V, Capacitor_SMD:C_1206_3216Metric, symbol Device:C
- added C26, C27, C29, C34: 10uF, Capacitor_SMD:C_0805_2012Metric, symbol Device:C
- added C28: 100nF, Capacitor_SMD:C_1206_3216Metric, symbol Device:C
- added C30, C36, C37: 2.2nF, Capacitor_SMD:C_0603_1608Metric, symbol Device:C
- added C31: 1nF, Capacitor_SMD:C_0603_1608Metric, symbol Device:C
- added C33: 270pF, Capacitor_SMD:C_0603_1608Metric, symbol Device:C
- added C38: 47uF 35V, Capacitor_SMD:CP_Elec_6.3x7.7, symbol Device:C_Polarized
- added C39: 100nF 50V, Capacitor_SMD:C_0603_1608Metric, symbol Device:C
- added C40: 2.2uF 50V, Capacitor_SMD:C_1210_3225Metric, symbol Device:C
- added D10, D11, D12, D14, D15: BAT54S, Package_TO_SOT_SMD:SOT-23, symbol Diode:BAT54S
- added D13: MAVI, LED_SMD:LED_0603_1608Metric, symbol Device:LED
- added D16: BZT52C18, Diode_SMD:D_SOD-123, symbol Device:D_Zener
- added D3: BZT52C3V3, Diode_SMD:D_SOD-123, symbol Device:D_Zener
- added D4, D6: BAT54C, Package_TO_SOT_SMD:SOT-23, symbol Diode:BAT54C
- added D5: BAT54WS, Diode_SMD:D_SOD-323, symbol Device:D_Schottky
- added D7: SS16, Diode_SMD:D_SMA, symbol Device:D_Schottky
- added D8: YESIL, LED_SMD:LED_0603_1608Metric, symbol Device:LED
- added D9: B5819W, Diode_SMD:D_SOD-123, symbol Device:D_Schottky
- added J2: ARM-SW (NC), Connector_JST:JST_XH_B2B-XH-A_1x02_P2.50mm_Vertical, symbol Connector_Generic:Conn_01x02
- added J3: PIEZO, Connector_JST:JST_XH_B2B-XH-A_1x02_P2.50mm_Vertical, symbol Connector_Generic:Conn_01x02
- added J4: HIDROFON, Connector_JST:JST_XH_B3B-XH-A_1x03_P2.50mm_Vertical, symbol Connector_Generic:Conn_01x03
- added J5: TRANSDUSOR, Connector_JST:JST_XH_B2B-XH-A_1x02_P2.50mm_Vertical, symbol Connector_Generic:Conn_01x02
- added J6: SIZINTI PROBU, Connector_JST:JST_XH_B2B-XH-A_1x02_P2.50mm_Vertical, symbol Connector_Generic:Conn_01x02
- added Q1: AO3401A, Package_TO_SOT_SMD:SOT-23, symbol Transistor_FET:AO3401A
- added Q2: 2N7002, Package_TO_SOT_SMD:SOT-23, symbol Transistor_FET:2N7002
- added R38: 100, Resistor_SMD:R_0603_1608Metric, symbol Device:R
- added R39: 62k, Resistor_SMD:R_0603_1608Metric, symbol Device:R
- added R40: 10k, Resistor_SMD:R_0603_1608Metric, symbol Device:R
- added R41: 47k, Resistor_SMD:R_0603_1608Metric, symbol Device:R
- added R42: 1k, Resistor_SMD:R_0603_1608Metric, symbol Device:R
- added R43: 330, Resistor_SMD:R_0603_1608Metric, symbol Device:R
- added R44: 1M, Resistor_SMD:R_0603_1608Metric, symbol Device:R
- added TP5: +3V3_AON, TestPoint:TestPoint_Pad_D1.5mm, symbol Connector:TestPoint
- added TP6: VREF_A, TestPoint:TestPoint_Pad_D1.5mm, symbol Connector:TestPoint
- added U1, U2: HT7533-1, Package_TO_SOT_SMD:SOT-89-3, symbol Regulator_Linear:HT75xx-1-SOT89
- added U10: DRV8871, Package_SO:Texas_HTSOP-8-1EP_3.9x4.9mm_P1.27mm_EP2.95x4.9mm_Mask2.4x3.1mm_ThermalVias, symbol Driver_Motor:DRV8871DDA
- added U3: MCP6042, Package_SO:SOIC-8_3.9x4.9mm_P1.27mm, symbol Amplifier_Operational:MCP6022
- added U4: TLV7031, Package_TO_SOT_SMD:SOT-23-5, symbol Comparator:TLV7031DBV
- added U5: LMR16006XDDCR, Package_TO_SOT_SMD:SOT-23-6, symbol Regulator_Switching:LMR16006YQ
- added U6: LP5907MFX-3.3, Package_TO_SOT_SMD:SOT-23-5, symbol Regulator_Linear:LP5907MFX-3.3
- added U7: Teensy 4.1, acoustic:Teensy4.1_Socket, symbol acoustic:Teensy4.1
- added U8, U9: MCP6022, Package_SO:SOIC-8_3.9x4.9mm_P1.27mm, symbol Amplifier_Operational:MCP6022
- C1: value 47uF 63V -> 47uF 35V; footprint Capacitor_SMD:CP_Elec_8x10 -> Capacitor_SMD:CP_Elec_6.3x7.7; MPN Panasonic EEE-FK1J470P -> Panasonic EEE-FK1V470P; Not Toplu giris kondansatoru (tether/aku kablosu rezonans sonum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 -> Toplu giris kondansatoru
- C11: value 100nF -> 10uF; footprint Capacitor_SMD:C_0603_1608Metric -> Capacitor_SMD:C_0805_2012Metric; MPN X7R 0603 16V -> X5R 0805 10V
- C13: footprint Capacitor_SMD:C_0603_1608Metric -> Capacitor_SMD:C_1206_3216Metric; MPN X7R 0603 16V -> C0G/NP0 1206 50V
- C14: value 100nF -> 1uF
- C2, C3: value 2.2uF 100V -> 2.2uF 50V; MPN X7R 1210 100V -> X7R 1210 50V
- C4: value 100nF 25V -> 100nF; MPN X7R 0603 25V -> X7R 0603 16V
- C5: value 22uF 10V -> 1uF 50V; MPN X7R 1206 10V -> X7R 1206 50V
- C6: value 22uF 10V -> 4.7uF; footprint Capacitor_SMD:C_1206_3216Metric -> Capacitor_SMD:C_0805_2012Metric; MPN X7R 1206 10V -> X5R 0805 10V
- C7: value 1uF -> 22uF 25V; footprint Capacitor_SMD:C_0603_1608Metric -> Capacitor_SMD:C_1210_3225Metric; MPN X7R 0603 16V -> X5R 1210 25V
- C8: value 1uF -> 100nF 50V; MPN X7R 0603 16V -> X7R 0603 50V
- C9: value 10uF -> 4.7uF
- D1: value SS16 -> SS26; MPN SS16 (60V 1A) -> SS26 (60V 2A)
- D2: value SMBJ30CA -> SMBJ20CA; MPN Littelfuse SMBJ30CA -> Littelfuse SMBJ20CA; Not Vrwm 30V; 6x ESC rejeneratif/enduktif sicrama kiskaci -> Vrwm 20V > 16.8V tam dolu; transdusor geri tepme kiskaci
- F1: value 1A 63V -> 2A 63V; MPN Littelfuse 0466001.NRHF -> Littelfuse 0466002.NRHF; Not Lojik + kontaktor bobini sigortasi -> Modem H-koprusu tepe akimi (ILIM 1 A) + lojik
- H1, H2, H3, H4: value CH3 -> M3; now left out of the parts list
- J1: value PIEZO/HV -> 4S LI-ION; Not 6S Li-Po girisi (ana sigortadan sonra, ESC kontaktorunden o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 -> 4S Li-ion paket (BMS dahili), 12.0 - 16.8 V
- L1: Not Isat >= 1 A gerekli -> Isat >= 1 A
- R10, R9: value 220 -> 10M; MPN 0603 220 1% -> 0603 10M 1%
- R11: value 100k -> 10M; MPN 0603 100k 1% -> 0603 10M 1%
- R12, R14: value 100k -> 1M; MPN 0603 100k 1% -> 0603 1M 1%
- R13, R15: value 100k -> 33k; MPN 0603 100k 1% -> 0603 33k 1%
- R16: value 100k -> 4.7M; MPN 0603 100k 1% -> 0603 4.7M 1%
- R17: value 4.7k -> 4.7M; MPN 0603 4.7k 1% -> 0603 4.7M 1%
- R18: value 4.7k -> 5.1M; MPN 0603 4.7k 1% -> 0603 5.1M 1%
- R19: value 33 -> 10k; MPN 0603 33 1% -> 0603 10k 1%
- R2: value 54.9k -> 100k; MPN 0603 54.9k 1% -> 0603 100k 1%
- R20: value 33 -> 1M; MPN 0603 33 1% -> 0603 1M 1%
- R21: value 10k -> 54.9k; MPN 0603 10k 1% -> 0603 54.9k 1%
- R23: value 10k -> 2.2k; MPN 0603 10k 1% -> 0603 2.2k 1%
- R24: value 47k -> 10k; MPN 0603 47k 1% -> 0603 10k 1%
- R25: value 1k -> 10k; MPN 0603 1k 1% -> 0603 10k 1%
- R26: value 68k -> 49.9; MPN 0603 68k 1% -> 0603 49.9 1%
- R27, R30: value 10k -> 1k; MPN 0603 10k 1% -> 0603 1k 1%
- R28: value 1k -> 10M; MPN 0603 1k 1% -> 0603 10M 1%
- R29: value 470 -> 9.1k; MPN 0603 470 1% -> 0603 9.1k 1%
- R3: value 10k -> 100; MPN 0603 10k 1% -> 0603 100 1%
- R31: value 10k -> 2.7k; MPN 0603 10k 1% -> 0603 2.7k 1%
- R32: value 47k -> 2.7k; MPN 0603 47k 1% -> 0603 2.7k 1%
- R33: value 10k -> 9.1k; MPN 0603 10k 1% -> 0603 9.1k 1%
- R36: value 100k -> 100; MPN 0603 100k 1% -> 0603 100 1%
- R37: value 330 -> 100; MPN 0603 330 1% -> 0603 100 1%
- R4: value 2.2k -> 100k; MPN 0603 2.2k 1% -> 0603 100k 1%
- R5: value 220 -> 100k; MPN 0603 220 1% -> 0603 100k 1%
- R6: value 220 -> 15k; MPN 0603 220 1% -> 0603 15k 1%
- R7: value 220 -> 1k; MPN 0603 220 1% -> 0603 1k 1%
- R8: value 220 -> 10k; MPN 0603 220 1% -> 0603 10k 1%
- TP1: value +24V -> VSYS; now left out of the parts list
- TP2, TP4: now left out of the parts list
- TP3: value +3V3 -> +3V3A; now left out of the parts list
Connections:
- net DEPTH_RAW is gone; now on net +5V: R21.1
- net IMU_SDA is gone; now on net GND: R20.2
- net T_ESC_EN is gone; now on net A_S1: R29.1
- net T_PWM1 is gone; now on net BATT_DIV: R6.1
- net T_PWM2 is gone; now on net BATT_DIV: R7.1
- net T_PWM5 is gone; now on net VREF_W: R10.1
- net +5V: now also R23.1, C22.1, C23.1, C24.1, D9.2 (A), U6.1 (IN), U6.3 (EN); no longer C12.1, C5.1, C6.1, C7.1, R2.1, R4.1
- net BATT_DIV: now also C4.1, R5.2, D3.1 (K); no longer C14.1, R26.2, R27.1, R28.1
- net BUCK_CB: now also C21.1, U5.1 (CB); no longer C4.1
- net BUCK_FB: now also R21.2, R22.1, U5.3 (FB); no longer R2.2, R3.1
- net BUCK_SW: now also C21.2, D7.1 (K), U5.6 (SW); no longer C4.2
- net GND: now also C4.2, R10.2, R18.2, R25.2, R4.2, R6.2, C16.2, C17.2, C18.2, C19.2, C20.2, C22.2, C23.2, C24.2, C25.2, C26.2, C27.2, C31.2, C32.2, C35.2, C36.2, C37.2, C38.2, C39.2, C41.2, D10.1 (A), D11.1 (A), D12.1 (A), D13.1 (K), D14.1 (A), D15.1 (A), D16.2 (A), D3.2 (A), D7.2 (A), D8.1 (K), J4.2 (Pin_2), J4.3 (Pin_3), Q2.2 (S), R39.2, R41.2, R44.2, U1.1 (GND), U10.1 (GND), U10.7 (GND), U10.9 (GND), U2.1 (GND), U3.4 (V-), U4.2 (V-), U5.2 (GND), U6.2 (GND), U7.1 (GND), U7.26 (GND), U7.39 (GND), U8.4 (V-), U9.4 (V-); no longer C13.2, C14.2, R11.2, R12.2, R13.2, R14.2, R15.2, R24.2, R27.2, R3.2, R30.2, R33.2, R36.2
- net LEAK_NODE: now also C41.1, J6.2 (Pin_2), R41.1, R42.1; no longer C13.1, R24.1, R25.1
- net LEAK_P: now also J6.1 (Pin_1), R40.2; no longer R23.2
- net LED_PWR_A: now also R23.2, D8.2 (A); no longer R4.2
- net LED_STAT_A: now also D13.2 (A), R43.2; no longer R37.2
- net TEENSY_VIN: now also D9.1 (K), U7.25 (VIN)
- net T_BATT_ADC: now also R7.2, U7.36 (15/A1); no longer R28.2
- net T_LEAK_ADC: now also R42.2, U7.37 (14/A0); no longer R25.2
- net T_LED: now also R43.1, U7.38 (13); no longer R37.1
- net VBAT_F: now also J2.1 (Pin_1); no longer D1.2 (A)
- net +24V renamed VSYS
- net VSYS: now also C5.1, C38.1, C39.1, Q1.2 (S), U1.2 (VIN), U10.5 (VM), U5.5 (VIN); no longer R26.1
- removed net +3V3: C8.1, C9.1, R17.1, R18.1, R23.1, TP3.1
- net BUCK_SHDN renamed BS_G
- net BS_G: now also R2.1, Q1.1 (G)
- net ESC_PWM0 renamed W_IN
- net W_IN: now also C13.2, U3.3 (+); no longer R5.2
- net ESC_PWM1 renamed W_A
- net W_A: now also U3.1, U3.5 (+); no longer R6.2
- net ESC_PWM2 renamed W_FB1
- net W_FB1: now also R12.2, U3.2 (-); no longer R7.2
- net ESC_PWM3 renamed T_HARV_PG
- net T_HARV_PG: now also U7.14 (12); no longer R14.1
- net ESC_PWM4 renamed VREF_W
- net VREF_W: now also C12.1, C14.2, R11.2, C15.2; no longer R15.1
- net ESC_PWM5 renamed W_ENV
- net W_ENV: now also C17.1, D5.1 (K), U4.3 (+); no longer R10.2
- net IMU_SCL renamed T_WAKE
- net T_WAKE: now also U7.30 (21/A7)
- removed net KILL_DIV: R32.2, R33.1, R34.1
- net KILL_RET renamed A_S1
- net A_S1: now also U8.1; no longer R32.1
- net LED_ESC_A renamed A_SK1
- net A_SK1: now also R32.1, C30.1
- net Q1_G renamed AFE_HI
- net AFE_HI: now also R33.1, C33.1, U9.1; no longer R35.2
- net Q2_B renamed A_FB1
- net A_FB1: now also U8.2 (-)
- net T_BUZZER renamed AFE_LO
- net AFE_LO: now also C30.2, U8.6 (-), U8.7, U9.3 (+)
- removed net T_DEPTH_ADC: C11.1, R21.2, R22.1
- net T_KILL_SENSE renamed A_G2
- net A_G2: now also C34.1
- net T_PWM0 renamed BATT_SW
- net BATT_SW: now also Q1.3 (D)
- net T_PWM3 renamed V_HARV
- net V_HARV: now also C9.1, D4.2, R44.1, U2.3 (VOUT)
- net T_PWM4 renamed +3V3_AON
- net +3V3_AON: now also C11.1, R17.1, C16.1, C19.1, D4.3, TP5.1, U3.8 (V+), U4.5 (V+)
- net T_SCL0 renamed WAKE_CMP
- net WAKE_CMP: now also D6.1, U4.1; no longer R17.2
- net T_SDA0 renamed BUCK_EN
- net BUCK_EN: now also C20.1, D6.3, U5.4 (~{SHDN}); no longer R18.2
- new net +3V3A: C25.1, C32.1, C35.1, D10.2 (K), D11.2 (K), D12.2 (K), R24.1, R40.1, TP3.1, U6.5 (OUT), U8.8 (V+), U9.8 (V+)
- new net +3V3_LDO: C6.1, D4.1, U1.3 (VOUT)
- new net ARM_RET: D1.2 (A), J2.2 (Pin_2)
- new net A_FB2: C33.2, R33.2, R34.1, U9.2 (-)
- new net A_G1: C29.1, R30.2
- new net A_IN: C28.2, R27.1
- new net A_INP: D10.3 (COM), R27.2, R28.1, U8.3 (+)
- new net A_SK2: C31.1, R32.2, U8.5 (+)
- new net BS_D: Q2.3 (D), R2.2
- new net BS_EN_G: Q2.1 (G), R3.2, R4.1
- new net HV_STORE: C7.1, C8.1, D14.2 (K), D15.2 (K), D16.1 (K), U2.2 (VIN)
- new net HYD_SIG: C13.1, C28.1, J4.1 (Pin_1)
- new net PZ1: D14.3 (COM), J3.1 (Pin_1)
- new net PZ2: D15.3 (COM), J3.2 (Pin_2)
- new net TX_ILIM: R39.1, U10.4 (ILIM)
- new net TX_IN1: R37.2, U10.3 (IN1)
- new net TX_IN2: R38.2, U10.2 (IN2)
- new net TX_OUT1: C40.1, U10.6 (OUT1)
- new net TX_OUT2: J5.2 (Pin_2), U10.8 (OUT2)
- new net TX_P: C40.2, J5.1 (Pin_1)
- new net T_ADC_HI: C37.1, D12.3 (COM), R36.2, U7.34 (17/A3)
- new net T_ADC_LO: C36.1, D11.3 (COM), R35.2, U7.35 (16/A2)
- new net T_BATT_EN: R3.1, U7.29 (22)
- new net T_PWR_HOLD: D6.2, U7.28 (23)
- new net T_TX_IN1: R37.1, U7.8 (6)
- new net T_TX_IN2: R38.1, U7.11 (9)
- new net VREF_A: C27.1, C29.2, C34.2, R26.2, R28.2, TP6.1
- new net VREF_BUF: R26.1, U9.6 (-), U9.7
- new net VREF_DIV: C26.1, R24.2, R25.1, U9.5 (+)
- new net W_B: D5.2 (A), R14.1, U3.7
- new net W_FB2: R14.2, R15.1, U3.6 (-)
- new net W_G1: C14.1, R13.2
- new net W_G2: C15.1, R15.2
- new net W_TH: C18.1, R17.2, R18.1, U4.4 (-)
- no-connect marks 35 -> 33
Other:
- note added: "Akustik modem vericisi (DRV8871, 24/28 kHz BFSK)"
- note added: "Anahtarli pil gerilim olcumu (uykuda 0 akim)"
- note added: "Analog besleme (LP5907 3.3 V)"
- note added: "Hep acik besleme: HT7533-1 + piezo hasadi (kopru + HT7533-1)"
- note added: "Hidrofon AFE: 20/40 dB cift kazanc, 40 kHz Sallen-Key"
- note added: "Pasif akustik uyanma (MCP6042 + TLV7031)"
- note added: "Pil girisi, kurma anahtari ve koruma (4S Li-ion)"
- note added: "Su sizinti probu ve durum LED"
- note added: "Teensy 4.1 (192 kHz cift ADC DMA, DSP)"
- note added: "Uyanma mandali (WAKE_CMP | PWR_HOLD -> BUCK_EN)"
- note added: "VSYS -> 5 V buck (LMR16006X, 700 kHz)"
- note removed: "5 V -> 3.3 V LDO ve Teensy VIN izolasyonu"
- note removed: "6S -> 5 V buck (LMR16006X, 700 kHz)"
- note removed: "6x Itici ESC PWM cikislari (M0..M5)"
- note removed: "Akustik buzzer ve durum LED"
- note removed: "Guc girisi ve koruma (6S Li-Po 22.2 V)"
- note removed: "Hidrostatik basinc sensoru (SEN0257 5V -> 3.3V ADC)"
- note removed: "IMU (AFE-I2C, I2C0 400 kHz)"
- note removed: "Su gecirmez manyetik kill-switch ve ESC guc kontaktoru"
- note removed: "Teensy 4.1 (Gercek Zamanli I/O)"
- note removed: "Tup ici su sizinti probu ve 6S batarya ADC bolucu"
- company: CU AVTECH — Stingray Sualti Sistemleri -> Pasif sonar + piezo enerji hasadi + akustik BFSK modem
- title: Akustik Suru Dugum Karti -> Akustik Suru Dugumu (acoustic-swarm-node)
